File: display.kicad_sch (KiCad schematic)
At the start: 20 parts, among them Q1 BC547, Q2 BC547, Q3 BC547, Q4 BC547, U1 SC39-11GWA, U2 SC39-11GWA, U3 SC39-11GWA, U4 SC39-11GWA

Commit message: reset annotations
Parts:
- renumbered R1 to R10, R2 to R11, R3 to R12, R4 to R13, R5 to R14, R6 to R15, R7 to R16, R8 to R17, R10 to R18, R11 to R19, R12 to R20, U1 to U4, U2 to U5, U3 to U6, U4 to U7
Changed lines of the file:
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@@
 		(on_board yes)
 		(dnp no)
-		(property "Reference" "R4"
+		(property "Reference" "R13"
 			(at 45.72 47.62 90)
 			(effects
@@
 			(project "display"
 				(path "/68f2073a-7618-4fa5-a11d-b71bb4f75794/260345d3-423b-4cc1-8385-8e7df36d7228"
-					(reference "R4")
+					(reference "R13")
 					(unit 1)
 				)
@@
 		(on_board yes)
 		(dnp no)
-		(property "Reference" "R1"
+		(property "Reference" "R10"
 			(at 45.72 28.57 90)
 			(effects
@@
 			(project "display"
 				(path "/68f2073a-7618-4fa5-a11d-b71bb4f75794/260345d3-423b-4cc1-8385-8e7df36d7228"
-					(reference "R1")
+					(reference "R10")
 					(unit 1)
 				)
@@
 		(on_board yes)
 		(dnp no)
-		(property "Reference" "R3"
+		(property "Reference" "R12"
 			(at 45.72 41.27 90)
 			(effects
@@
 			(project "display"
 				(path "/68f2073a-7618-4fa5-a11d-b71bb4f75794/260345d3-423b-4cc1-8385-8e7df36d7228"
-					(reference "R3")
+					(reference "R12")
 					(unit 1)
 				)
@@
 		(on_board yes)
 		(dnp no)
-		(property "Reference" "#PWR04"
+		(property "Reference" "#PWR023"
 			(at 182.88 113.03 0)
 			(effects
@@
 			(project "display"
 				(path "/68f2073a-7618-4fa5-a11d-b71bb4f75794/260345d3-423b-4cc1-8385-8e7df36d7228"
-					(reference "#PWR04")
+					(reference "#PWR023")
 					(unit 1)
 				)
@@
 		(on_board yes)
 		(dnp no)
-		(property "Reference" "R7"
+		(property "Reference" "R16"
 			(at 45.72 66.67 90)
 			(effects
@@
 			(project "display"
 				(path "/68f2073a-7618-4fa5-a11d-b71bb4f75794/260345d3-423b-4cc1-8385-8e7df36d7228"
-					(reference "R7")
+					(reference "R16")
 					(unit 1)
 				)
@@
 		(on_board yes)
 		(dnp no)
-		(property "Reference" "#PWR02"
+		(property "Reference" "#PWR021"
 			(at 96.52 113.03 0)
 			(effects
@@
 			(project "display"
 				(path "/68f2073a-7618-4fa5-a11d-b71bb4f75794/260345d3-423b-4cc1-8385-8e7df36d7228"
-					(reference "#PWR02")
+					(reference "#PWR021")
 					(unit 1)
 				)
@@
 		(on_board yes)
 		(dnp no)
-		(property "Reference" "#PWR01"
+		(property "Reference" "#PWR020"
 			(at 53.34 113.03 0)
 			(effects
@@
 			(project "display"
 				(path "/68f2073a-7618-4fa5-a11d-b71bb4f75794/260345d3-423b-4cc1-8385-8e7df36d7228"
-					(reference "#PWR01")
+					(reference "#PWR020")
 					(unit 1)
 				)
@@
 		(on_board yes)
 		(dnp no)
-		(property "Reference" "R12"
+		(property "Reference" "R20"
 			(at 170.18 97.15 90)
 			(effects
@@
 			(project "display"
 				(path "/68f2073a-7618-4fa5-a11d-b71bb4f75794/260345d3-423b-4cc1-8385-8e7df36d7228"
-					(reference "R12")
+					(reference "R20")
 					(unit 1)
 				)
@@
 		(on_board yes)
 		(dnp no)
-		(property "Reference" "#PWR03"
+		(property "Reference" "#PWR022"
 			(at 139.7 113.03 0)
 			(effects
@@
 			(project "display"
 				(path "/68f2073a-7618-4fa5-a11d-b71bb4f75794/260345d3-423b-4cc1-8385-8e7df36d7228"
-					(reference "#PWR03")
+					(reference "#PWR022")
 					(unit 1)
 				)
@@
 		(on_board yes)
 		(dnp no)
-		(property "Reference" "R8"
+		(property "Reference" "R17"
 			(at 45.72 73.02 90)
 			(effects
@@
 			(project "display"
 				(path "/68f2073a-7618-4fa5-a11d-b71bb4f75794/260345d3-423b-4cc1-8385-8e7df36d7228"
-					(reference "R8")
+					(reference "R17")
 					(unit 1)
 				)
@@
 		(on_board yes)
 		(dnp no)
-		(property "Reference" "R11"
+		(property "Reference" "R19"
 			(at 127 97.15 90)
 			(effects
@@
 			(project "display"
 				(path "/68f2073a-7618-4fa5-a11d-b71bb4f75794/260345d3-423b-4cc1-8385-8e7df36d7228"
-					(reference "R11")
+					(reference "R19")
 					(unit 1)
 				)
@@
 		(on_board yes)
 		(dnp no)
-		(property "Reference" "R5"
+		(property "Reference" "R14"
 			(at 45.72 53.97 90)
 			(effects
@@
 			(project "display"
 				(path "/68f2073a-7618-4fa5-a11d-b71bb4f75794/260345d3-423b-4cc1-8385-8e7df36d7228"
-					(reference "R5")
+					(reference "R14")
 					(unit 1)
 				)
@@
 		(on_board yes)
 		(dnp no)
-		(property "Reference" "R10"
+		(property "Reference" "R18"
 			(at 83.82 97.15 90)
 			(effects
@@
 			(project "display"
 				(path "/68f2073a-7618-4fa5-a11d-b71bb4f75794/260345d3-423b-4cc1-8385-8e7df36d7228"
-					(reference "R10")
+					(reference "R18")
 					(unit 1)
 				)
@@
 		(on_board yes)
 		(dnp no)
-		(property "Reference" "R2"
+		(property "Reference" "R11"
 			(at 45.72 34.92 90)
 			(effects
@@
 			(project "display"
 				(path "/68f2073a-7618-4fa5-a11d-b71bb4f75794/260345d3-423b-4cc1-8385-8e7df36d7228"
-					(reference "R2")
+					(reference "R11")
 					(unit 1)
 				)
@@
 		(on_board yes)
 		(dnp no)
-		(property "Reference" "U1"
+		(property "Reference" "U4"
 			(at 74.93 31.75 0)
 			(effects
@@
 			(project "display"
 				(path "/68f2073a-7618-4fa5-a11d-b71bb4f75794/260345d3-423b-4cc1-8385-8e7df36d7228"
-					(reference "U1")
+					(reference "U4")
 					(unit 1)
 				)
@@
 		(on_board yes)
 		(dnp no)
-		(property "Reference" "U2"
+		(property "Reference" "U5"
 			(at 113.03 31.75 0)
 			(effects
@@
 			(project "display"
 				(path "/68f2073a-7618-4fa5-a11d-b71bb4f75794/260345d3-423b-4cc1-8385-8e7df36d7228"
-					(reference "U2")
+					(reference "U5")
 					(unit 1)
 				)
@@
 		(on_board yes)
 		(dnp no)
-		(property "Reference" "R6"
+		(property "Reference" "R15"
 			(at 45.72 60.32 90)
 			(effects
@@
 			(project "display"
 				(path "/68f2073a-7618-4fa5-a11d-b71bb4f75794/260345d3-423b-4cc1-8385-8e7df36d7228"
-					(reference "R6")
+					(reference "R15")
 					(unit 1)
 				)
@@
 		(on_board yes)
 		(dnp no)
-		(property "Reference" "U4"
+		(property "Reference" "U7"
 			(at 189.23 31.75 0)
 			(effects
@@
 			(project "display"
 				(path "/68f2073a-7618-4fa5-a11d-b71bb4f75794/260345d3-423b-4cc1-8385-8e7df36d7228"
-					(reference "U4")
+					(reference "U7")
 					(unit 1)
 				)
@@
 		(on_board yes)
 		(dnp no)
-		(property "Reference" "U3"
+		(property "Reference" "U6"
 			(at 151.13 31.75 0)
 			(effects
@@
 			(project "display"
 				(path "/68f2073a-7618-4fa5-a11d-b71bb4f75794/260345d3-423b-4cc1-8385-8e7df36d7228"
-					(reference "U3")
-					(unit 1)
-				)
+					(reference "U6")
+					(unit 1)
+				)
